File: HUB0402.kicad_pcb (KiCad board)
At the start: 4 copper layers, 179 parts, among them U1 TLV75533PDBVR, U10 UPD350A/Q8X, U2 TLV62084DSGR, U3 SN74LVC1G14DCKR, U5 SN74LVC1G14DCKR, U7 UPD350A/Q8X, U8 UPD350A/Q8X

Commit message: Starting Layout
Parts:
- removed C13, C14, C15, C16, C17, C18, C19, C20, C21, C22, C23, C24, C26, C27, C28, C29, C30, C31, C43, C44, C48, C51, C52, C55, C63, C66, C67, C70: 0.1uF, Capacitor_SMD:C_0402_1005Metric
- removed C25, C32: 10pF, Capacitor_SMD:C_0402_1005Metric
- removed C3: NC, Capacitor_SMD:C_0402_1005Metric
- removed C42, C45, C50, C53, C65, C68: 1uF, Capacitor_SMD:C_0402_1005Metric
- removed C46, C49, C54, C64, C69: 2.2uF, Capacitor_SMD:C_0402_1005Metric
- removed C47, C56, C57, C62, C71, C72: 47uF, Capacitor_SMD:C_0805_2012Metric
- removed D1, D2, D3: BAV99, Package_TO_SOT_SMD:SOT-23
- removed JP1: SolderJumper_3_Open, Jumper:SolderJumper-3_P2.0mm_Open_TrianglePad1.0x1.5mm
- removed LED1, LED11, LED13, LED2, LED7: LED_Green, LED_SMD:LED_0603_1608Metric
- removed LED10, LED12, LED6: LED_Yellow, LED_SMD:LED_0603_1608Metric
- removed LED4, LED9: LED_Red, LED_SMD:LED_0603_1608Metric
- removed LED8: LED_Blue, LED_SMD:LED_0603_1608Metric
- removed R1, R36, R37, R38, R41, R55, R61, R75, R81: 1K, Resistor_SMD:R_0402_1005Metric
- removed R20, R27: 200K, Resistor_SMD:R_0402_1005Metric
- removed R21, R33, R34, R39, R40, R43, R44, R48, R50, R51, R53, R54, R56, R57, R59, R60, R63, R64, R65, R68, R70, R71, R73, R74, R77, R78, R79, R80: 100K, Resistor_SMD:R_0402_1005Metric
- removed R22, R23, R24, R25, R29, R47, R67: 10K, Resistor_SMD:R_0402_1005Metric
- removed R26: 12K, Resistor_SMD:R_0402_1005Metric
- removed R28, R52, R72: 90.9K, Resistor_SMD:R_0402_1005Metric
- removed R30: 24K, Resistor_SMD:R_0402_1005Metric
- removed R31: 40.2K, Resistor_SMD:R_0402_1005Metric
- removed R32: 3.83K, Resistor_SMD:R_0402_1005Metric
- removed R35, R46, R49, R66, R69: 0R, Resistor_SMD:R_0402_1005Metric
- removed R42, R62: 6.65K, Resistor_SMD:R_0402_1005Metric
- removed R45: 0R, Resistor_SMD:R_1210_3225Metric
- removed R58, R76: 2.2K, Resistor_SMD:R_0402_1005Metric
- removed TP1, TP2, TP3, TP4, TP5: TestPoint, TestPoint:TestPoint_Pad_D1.5mm
- removed U10, U7, U8: UPD350A/Q8X, Package_DFN_QFN:QFN-28-1EP_4x4mm_P0.4mm_EP2.4x2.4mm_ThermalVias
- removed U3, U5: SN74LVC1G14DCKR, Package_TO_SOT_SMD:SOT-353_SC-70-5
- added C10: 0.1uF, Capacitor_SMD:C_0402_1005Metric, F.Cu at (81.9, 84.9)
- added C77: 0.1uF, Capacitor_SMD:C_0402_1005Metric, F.Cu at (87.6, 84.9)
- added C78: 0.1uF, Capacitor_SMD:C_0402_1005Metric, F.Cu at (87.6, 86.8)
- added C79: 0.1uF, Capacitor_SMD:C_0402_1005Metric, F.Cu at (87.6, 88.8)
- added C80: 0.1uF, Capacitor_SMD:C_0402_1005Metric, F.Cu at (87.6, 90.8)
- added C81: 0.1uF, Capacitor_SMD:C_0402_1005Metric, F.Cu at (90.5, 77.0)
- added C82: 0.1uF, Capacitor_SMD:C_0402_1005Metric, F.Cu at (90.5, 79.0)
- added C83: 0.1uF, Capacitor_SMD:C_0402_1005Metric, F.Cu at (90.5, 80.9)
- added C84: 0.1uF, Capacitor_SMD:C_0402_1005Metric, F.Cu at (90.5, 82.9)
- added C85: 0.1uF, Capacitor_SMD:C_0402_1005Metric, F.Cu at (90.5, 84.9)
- added C86: 0.1uF, Capacitor_SMD:C_0402_1005Metric, F.Cu at (90.5, 86.8)
- added C87: 0.1uF, Capacitor_SMD:C_0402_1005Metric, F.Cu at (90.5, 88.8)
- added C88: 0.1uF, Capacitor_SMD:C_0402_1005Metric, F.Cu at (90.5, 90.8)
- added C89: 0.1uF, Capacitor_SMD:C_0402_1005Metric, F.Cu at (93.3, 77.0)
- added C90: 0.1uF, Capacitor_SMD:C_0402_1005Metric, F.Cu at (93.3, 79.0)
- added C91: 0.1uF, Capacitor_SMD:C_0402_1005Metric, F.Cu at (93.3, 80.9)
- added C92: 0.1uF, Capacitor_SMD:C_0402_1005Metric, F.Cu at (93.3, 82.9)
- added C93: 0.1uF, Capacitor_SMD:C_0402_1005Metric, F.Cu at (93.3, 84.9)
- added J3: 12401598E4_2A, footprints:TYPE-C-SMD_918-418K2022Y40003, F.Cu at (100.1, 56.9)
- added J4: 12401598E4_2A, footprints:TYPE-C-SMD_918-418K2022Y40003, F.Cu at (126.1, 62.9)
- added J5: 12401598E4_2A, footprints:TYPE-C-SMD_918-418K2022Y40003, F.Cu at (74.1, 62.9)
- added R10: 1K, Resistor_SMD:R_0402_1005Metric, F.Cu at (168.8, 63.5)
- added R6: 43k, Resistor_SMD:R_0603_1608Metric, F.Cu at (92.6, 56.6)
- added R7: 49.9k, Resistor_SMD:R_0603_1608Metric, F.Cu at (91.8, 59.0)
- added R8: 1K, Resistor_SMD:R_0402_1005Metric, F.Cu at (165.9, 69.5)
- added R9: 1K, Resistor_SMD:R_0402_1005Metric, F.Cu at (168.8, 61.5)
- added SW2: SW_Push, footprints:SW4_KMR221GLFS_CNK, F.Cu at (157.6, 71.6)
- added U4: USB7002T-I/KDX, Package_DFN_QFN:VQFN-100-1EP_12x12mm_P0.4mm_EP8x8mm, B.Cu at (86.8, 62.2)
- added XTAL2: 25MHz, Crystal:Crystal_SMD_Abracon_ABM8G-4Pin_3.2x2.5mm, B.Cu at (97.2, 65.9)
- C11: value 0.1uF -> 2.2u; footprint Capacitor_SMD:C_0402_1005Metric -> Capacitor_SMD:C_0603_1608Metric
- C12, C8: value 0.1uF -> 100n; footprint Capacitor_SMD:C_0402_1005Metric -> Capacitor_SMD:C_0603_1608Metric
- C33, C34, C35, C36, C73, C74, C75, C76: moved to B.Cu
- C37: value 2.2uF -> 10uF; footprint Capacitor_SMD:C_0402_1005Metric -> Capacitor_SMD:C_0603_1608Metric
- C38: value 0.1uF -> 10uF; footprint Capacitor_SMD:C_0402_1005Metric -> Capacitor_SMD:C_0603_1608Metric
- C39: value 47uF -> 10pF; footprint Capacitor_SMD:C_0805_2012Metric -> Capacitor_SMD:C_0402_1005Metric; moved to B.Cu
- C40: value 0.1uF -> 10pF; moved to B.Cu
- C41: value 2.2uF -> 0.1uF
- R11: value 1K -> 100K
- R12: value 1K -> 12K
- R13: value 1K -> 49.9k; footprint Resistor_SMD:R_0402_1005Metric -> Resistor_SMD:R_0603_1608Metric
- R14: value 10K -> 43k; footprint Resistor_SMD:R_0402_1005Metric -> Resistor_SMD:R_0603_1608Metric
- R15: value 10K -> 49.9k; footprint Resistor_SMD:R_0402_1005Metric -> Resistor_SMD:R_0603_1608Metric
- R16: value 10R -> 200k
- R17, R19: value 10K -> 200k
- R18: value 200K -> 200k
- R5: value 1K -> 43k; footprint Resistor_SMD:R_0402_1005Metric -> Resistor_SMD:R_0603_1608Metric
- moved R17 118.8 mm to (171.7, 61.5)
- moved R18 118.8 mm to (171.7, 63.5)
- moved R19 118.8 mm to (171.7, 65.5)
- moved R11 116.9 mm to (168.8, 65.5)
- moved R12 116.9 mm to (168.8, 67.5)
- moved R16 115.1 mm to (168.8, 69.5)
- moved R15 110.3 mm to (164.7, 64.3)
- moved R5 110.3 mm to (160.7, 66.8)
- moved R14 110.2 mm to (164.7, 61.8)
- moved R13 110.1 mm to (164.7, 59.3)
- moved C8 88.0 mm to (156.7, 66.8)
- moved C12 87.3 mm to (160.7, 59.3)
- moved C41 72.6 mm to (144.6, 64.9)
- moved C38 56.2 mm to (133.9, 64.5)
- moved U1 52.5 mm to (64.3, 61.2)
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Connections:
- C11 pad 1: +3V3 -> Net-(U4B-VBUS_MON_UP)
- C12 pad 1: +3V3 -> Net-(U4A-DP1_VBUS_MON)
- C37 pad 1: Net-(J3-VBUS_A) -> +5V
- C38 pad 1: /VMON0 -> +5V
- C39 pad 1: +5V -> /XI
- C40 pad 1: +5V -> /XO
- C41 pad 1: GND -> /RST
- C41 pad 2: +3V3 -> GND
- C8 pad 1: +3V3 -> Net-(U4A-DP2_VBUS_MON)
- R11 pad 1: Net-(LED3-Pad2) -> /RST
- R11 pad 2: /SUSPEND_IND -> +3V3
- R12 pad 1: Net-(U5-Y) -> GND
- R13 pad 1: Net-(LED5-Pad2) -> GND
- R13 pad 2: /HOST_TYPE0 -> Net-(U4A-DP2_VBUS_MON)
- R14 pad 1: Net-(U6-SPI_CLK/GPIO4) -> Net-(U4A-DP1_VBUS_MON)
- R14 pad 2: +3V3 -> +5V
- R15 pad 1: Net-(U6-SPI_DO/GPIO5) -> GND
- R15 pad 2: +3V3 -> Net-(U4A-DP1_VBUS_MON)
- R16 pad 1: Net-(U6-SPI_DI/GPIO9/CFG_BC_EN) -> GND
- R16 pad 2: +3V3 -> Net-(U4A-PF20/CFG_NON_REM)
- R17 pad 1: /SMBDAT -> GND
- R17 pad 2: +3V3 -> Net-(U4A-PF22/CFG_BC_EN)
- R18 pad 2: Net-(U6-SPI_DI/GPIO9/CFG_BC_EN) -> Net-(U4A-CFG_STRAP1)
- R19 pad 1: /SMBCLK -> GND
- R19 pad 2: +3V3 -> Net-(U4A-CFG_STRAP2)
- R5 pad 1: Net-(U3-Y) -> Net-(U4A-DP2_VBUS_MON)
- R5 pad 2: Net-(LED2-K) -> +5V
- U1 pad 4: Net-(U1-NC) -> unconnected-(U1-NC-Pad4)
Routing:
- net /USB3RX_A0_N: track 0.00 -> 13.5 mm, vias 0 -> 1
- net /U0_CC2: track 0.00 -> 13.3 mm, vias 0 -> 2
- net /USB3RX_A0_P: track 0.00 -> 12.8 mm, vias 0 -> 1
- net /USB2P0_N: track 0.00 -> 12.3 mm, vias 0 -> 2
- net /USB2P0_P: track 0.00 -> 11.4 mm, vias 0 -> 2
- net /USB2P2_P: track 0.00 -> 11.1 mm, vias 0 -> 2
- net /USB2P2_N: track 0.00 -> 10.6 mm, vias 0 -> 1
- net /U0_CC1: track 0.00 -> 10.3 mm, vias 0 -> 2
- net /XO: track 0.00 -> 7.75 mm
- net Net-(J3-SSTXN1): track 0.00 -> 7.65 mm, vias 0 -> 1
- net Net-(J3-SSTXP1): track 0.00 -> 7.46 mm, vias 0 -> 1
- net /USB3RX_B0_N: track 0.00 -> 7.28 mm, vias 0 -> 2
- net /USB3RX_B0_P: track 0.00 -> 6.87 mm, vias 0 -> 2
- net /USB3TX_B0_P: track 0.00 -> 6.18 mm
- net /XI: track 0.00 -> 6.00 mm
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- added copper zone on In1.Cu, net GND
- added copper zone on In3.Cu, net GND
- added copper zone on In5.Cu, net GND
- added copper zone on In6.Cu, net GND
- added copper zone on F.Cu, net Net-(U4B-VBUS_MON_UP)
Other:
- board outline added: 60 x 20 mm
- copper layers 4 -> 8

Commit message: Layout mostly done
Parts:
- removed C41, C89: 0.1uF, Capacitor_SMD:C_0402_1005Metric
- removed SW2: SW_Push, footprints:SW4_KMR221GLFS_CNK
- C10, C58, C59, C60, C61, C77, C79, C80, C84, C85, C86, C88, R10, R16, R17, R18, R19, R8, R9: moved to B.Cu
- C11, C12, C37, C38, C8: footprint Capacitor_SMD:C_0603_1608Metric -> Capacitor_SMD:C_0402_1005Metric
- R13, R14, R15, R5, R6, R7: footprint Resistor_SMD:R_0603_1608Metric -> Resistor_SMD:R_0402_1005Metric
- moved R19 89.0 mm to (82.8, 69.8), turned to 90 degrees
- moved R18 88.2 mm to (83.8, 69.8), turned to 90 degrees
- moved R13 82.9 mm to (81.9, 62.9), turned to 180 degrees
- moved R9 81.8 mm to (87.4, 54.0), turned to -90 degrees
- moved R17 81.6 mm to (90.4, 54.5), turned to -90 degrees
- moved R8 81.0 mm to (86.4, 54.0), turned to -90 degrees
- moved R10 81.0 mm to (88.4, 54.0), turned to -90 degrees
- moved R16 80.9 mm to (89.4, 54.2), turned to -90 degrees
- moved R5 79.0 mm to (81.7, 64.4), turned to -90 degrees
- moved C8 76.8 mm to (79.9, 62.8), turned to 180 degrees
- moved R11 76.8 mm to (92.1, 67.0), turned to 180 degrees
- moved R12 76.6 mm to (92.2, 68.0), turned to 180 degrees
- moved R15 74.8 mm to (89.9, 67.0)
- moved R14 74.4 mm to (90.6, 68.5), turned to -90 degrees
- moved C12 71.7 mm to (89.6, 68.5), turned to -90 degrees
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Connections:
- net /RST renamed Net-(U4A-RBIAS)
Routing:
- net /USB3RX_B1_N: track 0.00 -> 49.8 mm, vias 0 -> 2
- net /USB3RX_B1_P: track 0.00 -> 49.2 mm, vias 0 -> 2
- net /USB3RX_A1_N: track 0.00 -> 47.1 mm, vias 0 -> 2
- net /USB3RX_A1_P: track 0.00 -> 46.4 mm, vias 0 -> 2
- net /USB2P1_N: track 0.00 -> 44.9 mm, vias 0 -> 1
- net /USB2P1_P: track 0.00 -> 44.4 mm, vias 0 -> 2
- net /P1_CC2: track 0.00 -> 44.1 mm, vias 0 -> 3
- net /USB3TX_B1_N: track 0.00 -> 43.5 mm, vias 0 -> 2
- net /P1_CC1: track 0.00 -> 42.8 mm, vias 0 -> 4
- net /USB3TX_B1_P: track 0.00 -> 42.5 mm, vias 0 -> 2
- net /USB3TX_A1_N: track 0.00 -> 38.2 mm
- net /USB3TX_A1_P: track 0.00 -> 37.8 mm
- net /P2_CC2: track 0.00 -> 12.4 mm
- net +3V3: track 0.00 -> 12.1 mm, vias 0 -> 2
- net +1V2: track 0.00 -> 9.54 mm, vias 0 -> 7
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- added copper zone on In4.Cu, net +1V2
- added copper zone on In2.Cu, net +3V3
- added copper zone on F.Cu, net +5V
- added copper zone on F.Cu, net Net-(U4A-DP1_VBUS_MON)
- added copper zone on F.Cu, net Net-(U4A-DP2_VBUS_MON)
Other:
- board text added: "USB-C 5Gbps Splitter Ensure Upstream Supply 3A@5V Author: Loren Ashfield"

Commit message: Update
Parts:
- added H1: MountingHole, MountingHole:MountingHole_2.2mm_M2, F.Cu at (72.7, 55.4)
- added H2: MountingHole, MountingHole:MountingHole_2.2mm_M2, F.Cu at (72.7, 70.3)
- added H3: MountingHole, MountingHole:MountingHole_2.2mm_M2, F.Cu at (127.6, 55.4)
- added H4: MountingHole, MountingHole:MountingHole_2.2mm_M2, F.Cu at (127.6, 70.3)
- added TP1: TestPoint, TestPoint:TestPoint_Pad_D1.5mm, F.Cu at (77.2, 71.5)
- added TP2: TestPoint, TestPoint:TestPoint_Pad_D1.5mm, F.Cu at (120.5, 71.5)
- added TP3: TestPoint, TestPoint:TestPoint_Pad_D1.5mm, F.Cu at (79.8, 71.5)
- added TP4: TestPoint, TestPoint:TestPoint_Pad_D1.5mm, F.Cu at (123.1, 71.5)
- moved C37 2.20 mm to (75.3, 57.8)
- moved C38 1.90 mm to (125.1, 57.8)
- moved C35 0.19 mm to (95.9, 55.7)
- moved C36 0.16 mm to (95.9, 54.7)
Routing:
- net Net-(U2-FB): track 0.00 -> 9.90 mm
- net GND: track 0.00 -> 8.50 mm, vias 44 -> 88
- net +1V2: track 9.54 -> 16.0 mm, vias 7 -> 24
- net +3V3: track 12.1 -> 17.3 mm, vias 2 -> 16
- net /P2_CC2: track 12.4 -> 8.72 mm, vias 1 -> 2
- net /XI: track 3.10 -> 6.00 mm
- net /USB2P0_N: track 12.3 -> 14.6 mm, vias 2 -> 3
- net Net-(U2-SW): track 0.00 -> 2.26 mm
- net /USB2P0_P: track 11.4 -> 13.3 mm
- net Net-(U2-PG): track 0.00 -> 1.42 mm
- net /P2_CC1: track 8.80 -> 7.87 mm
- net Net-(J5-SSTXP1): vias 2 -> 1
- net Net-(J5-SSTXN1): vias 2 -> 1
- net +5V: vias 1 -> 0
Other:
- board text added: "Saccade scME6 Capstone Upstream 3A@5V"
- board text removed: "USB-C 5Gbps Splitter Ensure Upstream Supply 3A@5V Author: Loren Ashfield"
