File: HUB0402.kicad_sch (KiCad schematic)
At the start: 189 parts, among them J3 USB4155-03-C_REVA, J4 12401598E4_2A, J5 12401598E4_2A, SW1 SW_Push, U1 TLV75533PDBVR, U10 UPD350A/Q8X, U11 MIC94041YFL-TR, U2 TLV62084DSGR, U3 SN74LVC1G14DCKR, U5 SN74LVC1G14DCKR, U6 USB5926CT_KD, U7 UPD350A/Q8X, U8 UPD350A/Q8X, U9 MIC94041YFL-TR

Commit message: Starting Layout
Parts:
- removed C13, C14, C15, C16, C17, C18, C19, C20, C21, C22, C23, C24, C26, C27, C28, C29, C30, C31, C43, C44, C48, C51, C52, C55, C63, C66, C67, C70: 0.1uF, Capacitor_SMD:C_0402_1005Metric, symbol Device:C
- removed C25, C32: 10pF, Capacitor_SMD:C_0402_1005Metric, symbol Device:C
- removed C3: NC, Capacitor_SMD:C_0402_1005Metric, symbol Device:C
- removed C42, C45, C50, C53, C65, C68: 1uF, Capacitor_SMD:C_0402_1005Metric, symbol Device:C
- removed C46, C49, C54, C64, C69: 2.2uF, Capacitor_SMD:C_0402_1005Metric, symbol Device:C
- removed C47, C56, C57, C62, C71, C72: 47uF, Capacitor_SMD:C_0805_2012Metric, symbol Device:C
- removed D1, D2, D3: BAV99, Package_TO_SOT_SMD:SOT-23, symbol Diode:BAV99
- removed J3: USB4155-03-C_REVA, USB4155_03_C:GCT_USB4155-03-C_REVA, symbol USB4155-03-C_REVA:USB4155-03-C_REVA
- removed JP1: SolderJumper_3_Open, Jumper:SolderJumper-3_P2.0mm_Open_TrianglePad1.0x1.5mm, symbol Jumper:SolderJumper_3_Open
- removed LED1, LED11, LED13, LED2, LED7: LED_Green, LED_SMD:LED_0603_1608Metric, symbol Device:LED
- removed LED10, LED12, LED6: LED_Yellow, LED_SMD:LED_0603_1608Metric, symbol Device:LED
- removed LED3, LED5: B2612UDNB20D000312U1930, B2612UDNB20D000312U1930:0606 Bi colour LED, symbol B2612UDNB20D000312U1930:Bi_Colour_0606_LED
- removed LED4, LED9: LED_Red, LED_SMD:LED_0603_1608Metric, symbol Device:LED
- removed LED8: LED_Blue, LED_SMD:LED_0603_1608Metric, symbol Device:LED
- removed R1, R36, R37, R38, R41, R55, R61, R75, R81: 1K, Resistor_SMD:R_0402_1005Metric, symbol Device:R
- removed R20, R27: 200K, Resistor_SMD:R_0402_1005Metric, symbol Device:R
- removed R21, R33, R34, R39, R40, R43, R44, R48, R50, R51, R53, R54, R56, R57, R59, R60, R63, R64, R65, R68, R70, R71, R73, R74, R77, R78, R79, R80: 100K, Resistor_SMD:R_0402_1005Metric, symbol Device:R
- removed R22, R23, R24, R25, R29, R47, R67: 10K, Resistor_SMD:R_0402_1005Metric, symbol Device:R
- removed R26: 12K, Resistor_SMD:R_0402_1005Metric, symbol Device:R
- removed R28, R52, R72: 90.9K, Resistor_SMD:R_0402_1005Metric, symbol Device:R
- removed R30: 24K, Resistor_SMD:R_0402_1005Metric, symbol Device:R
- removed R31: 40.2K, Resistor_SMD:R_0402_1005Metric, symbol Device:R
- removed R32: 3.83K, Resistor_SMD:R_0402_1005Metric, symbol Device:R
- removed R35, R46, R49, R66, R69: 0R, Resistor_SMD:R_0402_1005Metric, symbol Device:R
- removed R42, R62: 6.65K, Resistor_SMD:R_0402_1005Metric, symbol Device:R
- removed R45: 0R, Resistor_SMD:R_1210_3225Metric, symbol Device:R
- removed R58, R76: 2.2K, Resistor_SMD:R_0402_1005Metric, symbol Device:R
- removed SW1: SW_Push, 3x4x2:Tactile 3x4x2mm TS-A010, symbol Switch:SW_Push
- removed TP1, TP2, TP3, TP4, TP5: TestPoint, TestPoint:TestPoint_Pad_D1.5mm, symbol Connector:TestPoint
- removed U10, U7, U8: UPD350A/Q8X, Package_DFN_QFN:QFN-28-1EP_4x4mm_P0.4mm_EP2.4x2.4mm_ThermalVias, symbol UPD350A_Q8X:UPD350A_Q8X
- removed U11, U9: MIC94041YFL-TR, MIC94041YFL:MIC94041YFL, symbol MIC94041YFL:MIC94041YFL-TR
- removed U3, U5: SN74LVC1G14DCKR, Package_TO_SOT_SMD:SOT-353_SC-70-5, symbol SN74LVC1G14DCKR:SN74LVC1G14DCKR
- removed U6: USB5926CT_KD, USB5926CT_KD:QFN40P1200X1200X90-101N-D, symbol USB5926CT_KD:USB5926CT_KD
- removed XTAL1: 25MHz, VXM7_9013_25M0000000:VXM7_MCH, symbol VXM7-9013-25M0000000:VXM7-9013-25M0000000
- added C10, C77, C78, C79, C80, C81, C82, C83, C84, C85, C86, C87, C88, C89, C90, C91, C92, C93: 0.1uF, Capacitor_SMD:C_0402_1005Metric, symbol Device:C
- added J3: 12401598E4_2A, footprints:TYPE-C-SMD_918-418K2022Y40003, symbol 12401598E4_2A:12401598E4_2A
- added R10, R8, R9: 1K, Resistor_SMD:R_0402_1005Metric, symbol Device:R
- added R6: 43k, Resistor_SMD:R_0603_1608Metric, symbol Device:R
- added R7: 49.9k, Resistor_SMD:R_0603_1608Metric, symbol Device:R
- added SW2: SW_Push, footprints:SW4_KMR221GLFS_CNK, symbol Switch:SW_Push
- added U4: USB7002T-I/KDX, Package_DFN_QFN:VQFN-100-1EP_12x12mm_P0.4mm_EP8x8mm, symbol USB7002:USB7002T-I_KDX
- added XTAL2: 25MHz, Crystal:Crystal_SMD_Abracon_ABM8G-4Pin_3.2x2.5mm, symbol VXM7-9013-25M0000000:VXM7-9013-25M0000000
- C11: value 0.1uF -> 2.2u; footprint Capacitor_SMD:C_0402_1005Metric -> Capacitor_SMD:C_0603_1608Metric
- C12, C8: value 0.1uF -> 100n; footprint Capacitor_SMD:C_0402_1005Metric -> Capacitor_SMD:C_0603_1608Metric
- C37: value 2.2uF -> 10uF; footprint Capacitor_SMD:C_0402_1005Metric -> Capacitor_SMD:C_0603_1608Metric
- C38: value 0.1uF -> 10uF; footprint Capacitor_SMD:C_0402_1005Metric -> Capacitor_SMD:C_0603_1608Metric
- C39: value 47uF -> 10pF; footprint Capacitor_SMD:C_0805_2012Metric -> Capacitor_SMD:C_0402_1005Metric
- C40: value 0.1uF -> 10pF
- C41: value 2.2uF -> 0.1uF
- J4, J5: footprint 12401598E4_2A:AMPHENOL_12401598E4_2A -> footprints:TYPE-C-SMD_918-418K2022Y40003
- R11: value 1K -> 100K; JLCA Type Basic -> (none); LCSC Link https://www.lcsc.com/product-detail/Chip-Resistor-Surface-M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 -> (none); LCSC Part # C21190 -> (none); MFR.Part # 0603WAF1001T5E -> (none); Manufacturer UNI-ROYAL(Uniroyal Elec) -> (none); Package R0603 -> (none)
- R12: value 1K -> 12K; JLCA Type Basic -> (none); LCSC Link https://www.lcsc.com/product-detail/Chip-Resistor-Surface-M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 -> (none); LCSC Part # C21190 -> (none); MFR.Part # 0603WAF1001T5E -> (none); Manufacturer UNI-ROYAL(Uniroyal Elec) -> (none); Package R0603 -> (none)
- R13: value 1K -> 49.9k; footprint Resistor_SMD:R_0402_1005Metric -> Resistor_SMD:R_0603_1608Metric; JLCA Type Basic -> (none); LCSC Link https://www.lcsc.com/product-detail/Chip-Resistor-Surface-M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 -> (none); LCSC Part # C21190 -> (none); MFR.Part # 0603WAF1001T5E -> (none); Manufacturer UNI-ROYAL(Uniroyal Elec) -> (none); Package R0603 -> (none)
- R14: value 10K -> 43k; footprint Resistor_SMD:R_0402_1005Metric -> Resistor_SMD:R_0603_1608Metric
- R15: value 10K -> 49.9k; footprint Resistor_SMD:R_0402_1005Metric -> Resistor_SMD:R_0603_1608Metric
- R16: value 10R -> 200k; JLCA Type (none) -> Basic; LCSC Link (none) -> https://www.lcsc.com/product-detail/Chip-Resistor-Surface-M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; LCSC Part # (none) -> C21190; MFR.Part # (none) -> 0603WAF1001T5E; Manufacturer (none) -> UNI-ROYAL(Uniroyal Elec); Package (none) -> R0603
- R17, R19: value 10K -> 200k; JLCA Type (none) -> Basic; LCSC Link (none) -> https://www.lcsc.com/product-detail/Chip-Resistor-Surface-M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; LCSC Part # (none) -> C21190; MFR.Part # (none) -> 0603WAF1001T5E; Manufacturer (none) -> UNI-ROYAL(Uniroyal Elec); Package (none) -> R0603
- R18: value 200K -> 200k; JLCA Type (none) -> Basic; LCSC Link (none) -> https://www.lcsc.com/product-detail/Chip-Resistor-Surface-M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; LCSC Part # (none) -> C21190; MFR.Part # (none) -> 0603WAF1001T5E; Manufacturer (none) -> UNI-ROYAL(Uniroyal Elec); Package (none) -> R0603; now fitted
- R5: value 1K -> 43k; footprint Resistor_SMD:R_0402_1005Metric -> Resistor_SMD:R_0603_1608Metric; JLCA Type Basic -> (none); LCSC Link https://www.lcsc.com/product-detail/Chip-Resistor-Surface-M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 -> (none); LCSC Part # C21190 -> (none); MFR.Part # 0603WAF1001T5E -> (none); Manufacturer UNI-ROYAL(Uniroyal Elec) -> (none); Package R0603 -> (none)
Connections:
- net HOST_TYPE0 is gone; now on an unnamed net: R13.2
- net SMBCLK is gone; now on net GND: R19.1
- net SMBDAT is gone; now on net GND: R17.1
- net SUSPEND_IND is gone; now on net +3V3: R11.2
- net VBUS1 is gone; now on net +5V: J4.A4 (VBUS), J4.A9 (VBUS__1), J4.B4 (VBUS__2), J4.B9 (VBUS__3)
- net VBUS2 is gone; now on net +5V: J5.A4 (VBUS), J5.A9 (VBUS__1), J5.B4 (VBUS__2), J5.B9 (VBUS__3)
- net VMON0 is gone; now on net +5V: C38.1
- net +1V2: now also C78.1, C79.1, C82.1, C83.1, C86.1, C87.1, C90.1, C91.1, C93.1, U4.18 (VDD12), U4.25 (VDD12), U4.33 (VDD12), U4.41 (VDD12), U4.55 (VDD12), U4.78 (VDD12), U4.83 (VDD12), U4.9 (VDD12), U4.93 (VDD12)
- net +3V3: now also C10.1, C77.1, C80.1, C81.1, C84.1, C85.1, C88.1, C89.1, C92.1, R8.1, U4.14 (USB2DN_DP3/PRT_DIS_P3), U4.15 (USB2DN_DM3/PRT_DIS_M3), U4.26 (VDD33), U4.37 (USB2DN_DP4/PRT_DIS_P4), U4.38 (USB2DN_DM4/PRT_DIS_M4), U4.44 (VDD33), U4.53 (VDD33), U4.62 (VDD33), U4.67 (VDD33), U4.79 (VDD33), U4.86 (VDD33), U4.99 (VDD33); no longer C11.1, C12.1, C41.2, C8.1, R14.2, R15.2, R16.2, R17.2, R19.2
- net +5V: now also C37.1, R14.2, R5.2, J3.A4 (VBUS), J3.A9 (VBUS__1), J3.B4 (VBUS__2), J3.B9 (VBUS__3), R6.2; no longer C39.1, C40.1
- net GND: now also C41.2, R12.1, R13.1, R15.1, R16.1, C10.2, C77.2, C78.2, C79.2, C80.2, C81.2, C82.2, C83.2, C84.2, C85.2, C86.2, C87.2, C88.2, C89.2, C90.2, C91.2, C92.2, C93.2, J3.A1 (GND), J3.A12 (GND__1), J3.B1 (GND__2), J3.B12 (GND__3), J3.SH1 (SHIELD), J3.SH2 (SHIELD__1), J3.SH3 (SHIELD__2), J3.SH4 (SHIELD__3), R10.1, R7.1, R9.1, SW2.1, SW2.3, U4.101 (VSS), U4.24 (TESTEN), U4.96 (ATEST), XTAL2.2, XTAL2.4; no longer C41.1
- net P1_CC1: now also U4.12 (DP1_CC1)
- net P1_CC2: now also U4.13 (DP1_CC2)
- net P2_CC1: now also U4.27 (DP2_CC1)
- net P2_CC2: now also U4.28 (DP2_CC2)
- net RST: now also C41.1, R11.1, SW2.2, U4.100 (RBIAS)
- net U0_CC1: now also J3.A5 (CC1), U4.87 (CC1_UP)
- net U0_CC2: now also J3.B5 (CC2), U4.88 (CC2_UP)
- net USB2P0_N: now also J3.A7 (DN1), J3.B7 (DN2), U4.90 (USB2UP_DM)
- net USB2P0_P: now also J3.A6 (DP1), J3.B6 (DP2), U4.89 (USB2UP_DP)
- net USB2P1_N: now also U4.6 (USB2DN_DM1/PRT_DIS_M1)
- net USB2P1_P: now also U4.5 (USB2DN_DP1/PRT_DIS_P1)
- net USB2P2_N: now also U4.30 (USB2DN_DM2/PRT_DIS_M2)
- net USB2P2_P: now also U4.29 (USB2DN_DP2/PRT_DIS_P2)
- net USB3RX_A0_N: now also J3.B11 (SSRXP1), U4.95 (USB3UP_RXDMA)
- net USB3RX_A0_P: now also J3.B10 (SSRXN1), U4.94 (USB3UP_RXDPA)
- net USB3RX_A1_N: now also U4.11 (USB3DN_RXDM1A)
- net USB3RX_A1_P: now also U4.10 (USB3DN_RXDP1A)
- net USB3RX_A2_N: now also U4.35 (USB3DN_RXDM2A)
- net USB3RX_A2_P: now also U4.34 (USB3DN_RXDP2A)
- net USB3RX_B0_N: now also J3.A10 (SSRXN2), U4.85 (USB3UP_RXDMB)
- net USB3RX_B0_P: now also J3.A11 (SSRXP2), U4.84 (USB3UP_RXDPB)
- net USB3RX_B1_N: now also U4.20 (USB3DN_RXDM1B)
- net USB3RX_B1_P: now also U4.19 (USB3DN_RXDP1B)
- net USB3RX_B2_N: now also U4.43 (USB3DN_RXDM2B)
- net USB3RX_B2_P: now also U4.42 (USB3DN_RXDP2B)
- net USB3TX_A0_N: now also U4.92 (USB3UP_TXDMA)
- net USB3TX_A0_P: now also U4.91 (USB3UP_TXDPA)
- net USB3TX_A1_N: now also U4.8 (USB3DN_TXDM1A)
- net USB3TX_A1_P: now also U4.7 (USB3DN_TXDP1A)
- net USB3TX_A2_N: now also U4.32 (USB3DN_TXDM2A)
- net USB3TX_A2_P: now also U4.31 (USB3DN_TXDP2A)
- net USB3TX_B0_N: now also U4.82 (USB3UP_TXDMB)
- net USB3TX_B0_P: now also U4.81 (USB3UP_TXDPB)
- net USB3TX_B1_N: now also U4.17 (USB3DN_TXDM1B)
- net USB3TX_B1_P: now also U4.16 (USB3DN_TXDP1B)
- net USB3TX_B2_N: now also U4.40 (USB3DN_TXDM2B)
- net USB3TX_B2_P: now also U4.39 (USB3DN_TXDP2B)
- net at R5.1: now also C8.1, U4.36 (DP2_VBUS_MON)
- net at C33.1: now also J3.A2 (SSTXP1)
- net at R12.2: now also U4.1 (RESET_N)
- net at C34.1: now also J3.A3 (SSTXN1)
- net at C36.1: now also J3.B2 (SSTXP2)
- net at C35.1: now also J3.B3 (SSTXN2)
- net at R18.2: now also U4.21 (CFG_STRAP1); no longer R16.1
- net at R14.1: now also C12.1, R15.2, U4.4 (DP1_VBUS_MON)
- new net: R16.2, U4.69 (PF20/CFG_NON_REM)
- new net: R17.2, U4.70 (PF22/CFG_BC_EN)
- new net: R19.2, U4.22 (CFG_STRAP2)
- new net: R9.2, U4.64 (TEST2)
- new net: C11.1, R6.1, R7.2, U4.80 (VBUS_MON_UP)
- new net: R8.2, U4.63 (TEST1)
- new net: R10.2, U4.65 (TEST3)
- new net XI: C39.1, U4.98 (XTALI/CLK_IN), XTAL2.1
- new net XO: C40.1, U4.97 (XTALO), XTAL2.3
- no-connect marks 43 -> 34
Other:
- note added: "Oscillator"
- note added: "USB7002 Main"
- note added: "USB7002 Power"
- note added: "USB7002 USB"
- note removed: "DNP when using SPI flash"
- note removed: "Hub Controller"
- note removed: "Indicators"
- note removed: "USB-C Port 0"
- note removed: "USB-C Port 1"
- note removed: "USB-C Port 2"
- company: Jobit Joseph @ Semicon Media -> Author: Loren Ashfield
- title: USB 3.2 HUB -> USB-C 3.2 PD Splitter
- moved on the sheet: C1, C2, C33, C34, C35, C36, C4, C5, C58, C59, C6, C60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

Commit message: Layout mostly done
Parts:
- removed C41, C89: 0.1uF, Capacitor_SMD:C_0402_1005Metric, symbol Device:C
- removed SW2: SW_Push, footprints:SW4_KMR221GLFS_CNK, symbol Switch:SW_Push
- C11, C12, C37, C38, C8: footprint Capacitor_SMD:C_0603_1608Metric -> Capacitor_SMD:C_0402_1005Metric
- R13, R14, R15, R5, R6, R7: footprint Resistor_SMD:R_0603_1608Metric -> Resistor_SMD:R_0402_1005Metric
Connections:
- net RST: no longer names the net of R11.1, U4.100 (RBIAS)
Other:
- note added: "*Review 3v3"
- moved on the sheet: R11

Commit message: Update
Parts:
- added H1, H2, H3, H4: MountingHole, MountingHole:MountingHole_2.2mm_M2, symbol Mechanical:MountingHole
- added TP1, TP2, TP3, TP4: TestPoint, TestPoint:TestPoint_Pad_D1.5mm, symbol Connector:TestPoint
Connections:
- net +5V: now also TP1.1, TP2.1
- net GND: now also TP3.1, TP4.1
